File: pcb/zoom_pad.kicad_pcb (KiCad board)
At the start: 2 copper layers, 126 x 50 mm, 19 parts, among them J2 Conn_02x03_Counter_Clockwise, Q1 FDN340P, Q2 BSS123, SW1 RG_encoder_switch, U1 ESP32-WROOM-32D

Commit message: PCB v1.1
Parts:
- removed J2: Conn_02x03_Counter_Clockwise, Connector:Tag-Connect_TC2030-IDC-NL_2x03_P1.27mm_Vertical
- removed JP1: Jumper_2_Open, Jumper:SolderJumper-2_P1.3mm_Open_RoundedPad1.0x1.5mm
- added G***: LOGO, LOGO, F.Cu at (79.8, 94.5)
- added G***: LOGO, LOGO, F.Cu at (123.0, 91.5)
- added J1: Conn_02x03_Odd_Even, Connector:Tag-Connect_TC2030-IDC-NL_2x03_P1.27mm_Vertical, F.Cu at (63.0, 120.8)
- added S5: DD-15326, asl_footprints:sparkfun_tactile_color, F.Cu at (171.0, 120.8)
- moved SW1 39.6 mm to (162.0, 97.0)
- moved S4 18.5 mm to (147.0, 120.8)
- moved C1 16.0 mm to (164.5, 107.9)
- moved D1 16.0 mm to (169.0, 113.9)
- moved Q1 16.0 mm to (169.0, 109.4)
- moved Q2 16.0 mm to (164.5, 113.9)
- moved R1 16.0 mm to (164.5, 110.4)
- moved S3 14.2 mm to (123.0, 120.8)
- moved R4 12.9 mm to (159.5, 114.0), turned to 90 degrees
- moved R2 12.5 mm to (169.0, 105.9), turned to 0 degrees
- moved S2 9.86 mm to (99.0, 120.8)
- moved R3 6.49 mm to (159.5, 110.2), turned to -90 degrees
- moved S1 5.55 mm to (75.0, 120.8)
Connections:
- net Net-(U1-Pad3) renamed /EN
- BT1 pad 2: (no net) -> GND
- U1 pad 13: /TMS -> (no net)
- U1 pad 14: /TDI -> (no net)
- U1 pad 16: /TCK -> (no net)
- U1 pad 23: /TDO -> GND
- U1 pad 25: (no net) -> /IO0
- U1 pad 33: (no net) -> Net-(S5-Pad1)
- U1 pad 34: (no net) -> /RXDO
- U1 pad 35: (no net) -> /TXDO
- U1 pad 36: (no net) -> Net-(SW1-PadA)
- U1 pad 37: (no net) -> Net-(SW1-PadB)
- U1 pad 8: Net-(SW1-PadA) -> (no net)
- U1 pad 9: Net-(SW1-PadB) -> (no net)
Routing:
- net Net-(S5-Pad1): track 0.00 -> 105.9 mm, vias 0 -> 2
- net /EN: track 86.2 -> 141.5 mm
- net Net-(SW1-PadB): track 29.9 -> 81.0 mm, vias 0 -> 1
- net Net-(SW1-PadA): track 31.4 -> 82.0 mm, vias 0 -> 1
- net /GREEN_LED: track 46.6 -> 89.3 mm, vias 0 -> 1
- net /VIN: track 115.3 -> 156.2 mm, vias 4 -> 1
- net /RED_LED: track 46.9 -> 85.0 mm, vias 0 -> 1
- net /RXDO: track 0.00 -> 30.4 mm, vias 0 -> 1
- net /TXDO: track 0.00 -> 30.0 mm, vias 0 -> 1
- net /TMS: track 28.8 -> 0.00 mm
- net /TDO: track 24.9 -> 0.00 mm, vias 2 -> 0
- net /SW: track 42.5 -> 21.8 mm
- net /IO0: track 0.00 -> 19.6 mm, vias 0 -> 1
- net Net-(S4-Pad1): track 90.3 -> 71.6 mm
- net Net-(S3-Pad1): track 61.4 -> 46.3 mm
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Other:
- board text added: "Don't let Zoom control you!"
- board text added: "LEAVE"
- board text added: "Lustig Labworks - Dec 2020"
- board text added: "VIEW"
- board text added: "VOLUME"
- board text removed: "GALLERY"
- board text removed: "Lustig Labworks Dec 2020"
- board text removed: "VOL"
