File: pcb/zoom_pad.kicad_sch (KiCad schematic)
At the start: 20 parts, among them J2 Conn_02x03_Counter_Clockwise, Q1 FDN340P, Q2 BSS123, SW1 RG_encoder_switch, U1 ESP32-WROOM-32D

Commit message: PCB v1.1
Parts:
- removed BT2: 2463, Battery:BatteryHolder_Keystone_2466_1xAAA, symbol Device:Battery
- removed J2: Conn_02x03_Counter_Clockwise, Connector:Tag-Connect_TC2030-IDC-NL_2x03_P1.27mm_Vertical, symbol Connector_Generic:Conn_02x03_Counter_Clockwise
- removed JP1: Jumper_2_Open, Jumper:SolderJumper-2_P1.3mm_Open_RoundedPad1.0x1.5mm, symbol Jumper:Jumper_2_Open
- added J1: Conn_02x03_Odd_Even, Connector:Tag-Connect_TC2030-IDC-NL_2x03_P1.27mm_Vertical, symbol Connector_Generic:Conn_02x03_Odd_Even
- added S5: DD-15326, asl_footprints:sparkfun_tactile_color, symbol asl_symbols_new:B3F-4000
Connections:
- net TDO is gone; now on net GND: U1.23 (IO15)
- net GND: now also BT1.2 (-), J1.4 (Pin_4), S5.3 (out1), S5.4 (out2)
- net VIN: now also J1.2 (Pin_2)
- net EN: now reaches R2.1, U1.3 (EN)
- net EN: now also J1.1 (Pin_1)
- net at SW1.A: now also U1.36 (IO22); no longer U1.8 (IO32)
- net at SW1.B: now also U1.37 (IO23); no longer U1.9 (IO33)
- net IO0: now reaches U1.25 (IO0)
- net IO0: now also J1.6 (Pin_6)
- net at U1.33 (IO21): now also S5.1 (in1)
- net RXDO: now reaches U1.34 (RXD0/IO3)
- net RXDO: now also J1.5 (Pin_5)
- net TXDO: now reaches U1.35 (TXD0/IO1)
- net TXDO: now also J1.3 (Pin_3)
- net TCK: no longer names the net of U1.16 (IO13)
- net TDI: no longer names the net of U1.14 (IO12)
- net TMS: no longer names the net of U1.13 (IO14)
- no-connect marks 0 -> 23
Other:
- moved on the sheet: BT1, S1, S2, S3, S4, SW1
